Commit message: baxter config

File: src/baxter_moveit/baxter_moveit_config/config/baxter_base.srdf.xacro (robot description, xacro)
@@ -25,7 +25,11 @@
     <group name="left_hand">
         <chain base_link="left_hand" tip_link="$(arg left_tip_name)" />
+        <joint name="l_gripper_l_finger_joint" />
+        <passive_joint name="l_gripper_r_finger_joint" />
     </group>
     <group name="right_hand">
         <chain base_link="right_hand" tip_link="$(arg right_tip_name)" />
+        <joint name="r_gripper_l_finger_joint" />
+        <passive_joint name="r_gripper_r_finger_joint" />
     </group>
     <!--END EFFECTOR: Purpose: Represent information about an end effector.-->

Commit message: gripper almost

File: src/baxter_moveit/baxter_moveit_config/config/baxter_base.srdf.xacro (robot description, xacro)
@@ -26,10 +26,12 @@
         <chain base_link="left_hand" tip_link="$(arg left_tip_name)" />
         <joint name="l_gripper_l_finger_joint" />
-        <passive_joint name="l_gripper_r_finger_joint" />
+        <joint name="l_gripper_r_finger_joint" />
+        <!-- <passive_joint name="l_gripper_r_finger_joint" /> -->
     </group>
     <group name="right_hand">
         <chain base_link="right_hand" tip_link="$(arg right_tip_name)" />
         <joint name="r_gripper_l_finger_joint" />
-        <passive_joint name="r_gripper_r_finger_joint" />
+        <joint name="r_gripper_r_finger_joint" />
+        <!-- <passive_joint name="r_gripper_r_finger_joint" /> -->
     </group>
     <!--END EFFECTOR: Purpose: Represent information about an end effector.-->

Commit message: planit

File: src/baxter_moveit/baxter_moveit_config/config/baxter_base.srdf.xacro (robot description, xacro)
@@ -28,4 +28,6 @@
         <joint name="l_gripper_r_finger_joint" />
         <!-- <passive_joint name="l_gripper_r_finger_joint" /> -->
+        <link name="l_gripper_l_finger_tip" />
+        <link name="l_gripper_r_finger_tip" />
     </group>
     <group name="right_hand">
@@ -34,4 +36,6 @@
         <joint name="r_gripper_r_finger_joint" />
         <!-- <passive_joint name="r_gripper_r_finger_joint" /> -->
+        <link name="r_gripper_l_finger_tip" />
+        <link name="r_gripper_r_finger_tip" />
     </group>
     <!--END EFFECTOR: Purpose: Represent information about an end effector.-->
