Commit message: cylinder demo

File: src/baxter_moveit/baxter_moveit/urdf/baxter_base.urdf.xacro (robot description, xacro)
@@ -270,5 +270,5 @@
     <inertial>
       <origin rpy="0 0 0" xyz="0.01783 0.00086 0.19127"/>
-      <mass value="5.70044"/>
+      <mass value="1.70044"/>
       <inertia ixx="0.04709102262" ixy="0.00012787556" ixz="0.00614870039" iyy="0.03766976455" iyz="0.00078086899" izz="0.03595988478"/>
     </inertial>
@@ -292,5 +292,5 @@
     <inertial>
       <origin rpy="0 0 0" xyz="0.06845 0.00269 -0.00529"/>
-      <mass value="3.22698"/>
+      <mass value="1.22698"/>
       <inertia ixx="0.01175209419" ixy="-0.00030096398" ixz="0.00207675762" iyy="0.0278859752" iyz="-0.00018821993" izz="0.02078749298"/>
     </inertial>
@@ -314,5 +314,5 @@
     <inertial>
       <origin rpy="0 0 0" xyz="-0.00276 0.00132 0.18086"/>
-      <mass value="4.31272"/>
+      <mass value="1.31272"/>
       <inertia ixx="0.02661733557" ixy="0.00029270634" ixz="0.00392189887" iyy="0.02844355207" iyz="0.0010838933" izz="0.01248008322"/>
     </inertial>
@@ -349,5 +349,5 @@
     <inertial>
       <origin rpy="0 0 0" xyz="0.02611 0.00159 -0.01117"/>
-      <mass value="2.07206"/>
+      <mass value="1.07206"/>
       <inertia ixx="0.00711582686" ixy="0.00036036173" ixz="0.0007459496" iyy="0.01318227876" iyz="-0.00019663418" izz="0.00926852064"/>
     </inertial>
@@ -371,5 +371,5 @@
     <inertial>
       <origin rpy="0 0 0" xyz="-0.00168 0.0046 0.13952"/>
-      <mass value="2.24665"/>
+      <mass value="1.24665"/>
       <inertia ixx="0.01667742825" ixy="0.00018403705" ixz="0.00018657629" iyy="0.01675457264" iyz="-0.00064732352" izz="0.0037463115"/>
     </inertial>
@@ -413,5 +413,5 @@
     <inertial>
       <origin rpy="0 0 0" xyz="0.06041 0.00697 0.006"/>
-      <mass value="1.60979"/>
+      <mass value="0.60979"/>
       <inertia ixx="0.00387607152" ixy="-0.00044384784" ixz="-0.00021115038" iyy="0.00700537914" iyz="0.00015348067" izz="0.0055275524"/>
     </inertial>
@@ -638,5 +638,5 @@
     <inertial>
       <origin rpy="0 0 0" xyz="0.01783 0.00086 0.19127"/>
-      <mass value="5.70044"/>
+      <mass value="1.70044"/>
       <inertia ixx="0.04709102262" ixy="0.00012787556" ixz="0.00614870039" iyy="0.03766976455" iyz="0.00078086899" izz="0.03595988478"/>
     </inertial>
@@ -660,5 +660,5 @@
     <inertial>
       <origin rpy="0 0 0" xyz="0.06845 0.00269 -0.00529"/>
-      <mass value="3.22698"/>
+      <mass value="1.22698"/>
       <inertia ixx="0.01175209419" ixy="-0.00030096398" ixz="0.00207675762" iyy="0.0278859752" iyz="-0.00018821993" izz="0.02078749298"/>
     </inertial>
@@ -682,5 +682,5 @@
     <inertial>
       <origin rpy="0 0 0" xyz="-0.00276 0.00132 0.18086"/>
-      <mass value="4.31272"/>
+      <mass value="1.31272"/>
       <inertia ixx="0.02661733557" ixy="0.00029270634" ixz="0.00392189887" iyy="0.02844355207" iyz="0.0010838933" izz="0.01248008322"/>
     </inertial>
@@ -717,5 +717,5 @@
     <inertial>
       <origin rpy="0 0 0" xyz="0.02611 0.00159 -0.01117"/>
-      <mass value="2.07206"/>
+      <mass value="1.07206"/>
       <inertia ixx="0.00711582686" ixy="0.00036036173" ixz="0.0007459496" iyy="0.01318227876" iyz="-0.00019663418" izz="0.00926852064"/>
     </inertial>
@@ -739,5 +739,5 @@
     <inertial>
       <origin rpy="0 0 0" xyz="-0.00168 0.0046 0.13952"/>
-      <mass value="2.24665"/>
+      <mass value="1.24665"/>
       <inertia ixx="0.01667742825" ixy="0.00018403705" ixz="0.00018657629" iyy="0.01675457264" iyz="-0.00064732352" izz="0.0037463115"/>
     </inertial>
@@ -781,5 +781,5 @@
     <inertial>
       <origin rpy="0 0 0" xyz="0.06041 0.00697 0.006"/>
-      <mass value="1.60979"/>
+      <mass value="0.60979"/>
       <inertia ixx="0.00387607152" ixy="-0.00044384784" ixz="-0.00021115038" iyy="0.00700537914" iyz="0.00015348067" izz="0.0055275524"/>
     </inertial>
